File: H2AR30/Design/H2AR30.sch (EAGLE design)
At the start: 59 parts, among them P1 HEXABIT_17.32, U2 INA199A2DCKT, U3 INA199A2DCKT, U4 TEXAS_INSTRUMENTS_REF3212AIDB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, X1 XTALL_CSTCE8M00G52

Commit message: some bugs fixed
Parts:
- U2: value INA199A2DCKT -> INA199B2DCKT; MPN (none) -> INA199B2DCKT
- U3: value INA199A2DCKT -> INA199B2DCKT
Other:
- note added: "Current and Voltage Sense Module"
- note added: "H2AR3_backend"
- note removed: "RGB LED"
Changed lines of the file:
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@@
 <part name="P2" library="HEXABITZ_CONNECTION_PARTS" library_urn="urn:adsk.eagle:library:20064553" deviceset="1546111-2" device="" package3d_urn="urn:adsk.eagle:package:19666461/3"/>
 <part name="P3" library="HEXABITZ_CONNECTION_PARTS" library_urn="urn:adsk.eagle:library:20064553" deviceset="1546111-2" device="" package3d_urn="urn:adsk.eagle:package:19666461/3"/>
-<part name="U2" library="HEXABITZ_ICs" library_urn="urn:adsk.eagle:library:20064554" deviceset="INA199A2DCKT" device="" package3d_urn="urn:adsk.eagle:package:19904117/2"/>
+<part name="U2" library="HEXABITZ_ICs" library_urn="urn:adsk.eagle:library:20064554" deviceset="INA199A2DCKT" device="" package3d_urn="urn:adsk.eagle:package:19904117/2" value="INA199B2DCKT">
+<attribute name="MPN" value="INA199B2DCKT"/>
+</part>
 <part name="C10" library="HEXABITZ_RCLS" library_urn="urn:adsk.eagle:library:20064561" deviceset="C-0603" device="" package3d_urn="urn:adsk.eagle:package:19666468/2" value="10uF"/>
 <part name="C11" library="HEXABITZ_RCLS" library_urn="urn:adsk.eagle:library:20064561" deviceset="C-0603" device="" package3d_urn="urn:adsk.eagle:package:19666468/2" value="1uF"/>
@@
 <part name="R9" library="HEXABITZ_RCLS" library_urn="urn:adsk.eagle:library:20064561" deviceset="R_1206" device="R1206" package3d_urn="urn:adsk.eagle:package:23540/2" value="330k"/>
 <part name="R10" library="HEXABITZ_RCLS" library_urn="urn:adsk.eagle:library:20064561" deviceset="R_1206" device="R1206" package3d_urn="urn:adsk.eagle:package:23540/2" value="330k"/>
-<part name="U3" library="HEXABITZ_ICs" library_urn="urn:adsk.eagle:library:20064554" deviceset="INA199A2DCKT" device="" package3d_urn="urn:adsk.eagle:package:19904117/2"/>
+<part name="U3" library="HEXABITZ_ICs" library_urn="urn:adsk.eagle:library:20064554" deviceset="INA199A2DCKT" device="" package3d_urn="urn:adsk.eagle:package:19904117/2" value="INA199B2DCKT"/>
 <part name="C16" library="HEXABITZ_RCLS" library_urn="urn:adsk.eagle:library:20064561" deviceset="C-0603" device="" package3d_urn="urn:adsk.eagle:package:19666468/2" value="10uF"/>
 <part name="C17" library="HEXABITZ_RCLS" library_urn="urn:adsk.eagle:library:20064561" deviceset="C-0603" device="" package3d_urn="urn:adsk.eagle:package:19666468/2" value="1uF"/>
@@
 <text x="199.4662" y="19.6342" size="1.9304" layer="100" font="vector">Title</text>
 <text x="180.9242" y="19.6342" size="1.9304" layer="102" font="vector">H2AR3</text>
-<text x="179.2478" y="11.2014" size="1.9304" layer="101" font="vector">RGB LED</text>
-<text x="206.3242" y="19.6342" size="1.9304" layer="101" font="vector">H2AR3_Frontend</text>
+<text x="206.3242" y="19.6342" size="1.9304" layer="101" font="vector">H2AR3_backend</text>
 <wire x1="168.91" y1="3.81" x2="168.91" y2="8.128" width="0.1524" layer="205"/>
 <wire x1="168.91" y1="8.128" x2="168.91" y2="18.288" width="0.1524" layer="205"/>
@@
 <text x="30.48" y="198.12" size="1.778" layer="150">VDD=3.3 Volts</text>
 <text x="183.8778" y="4.9414" size="1.9304" layer="101" font="vector">Amir_Tabbakh</text>
+<text x="170.3578" y="11.2014" size="1.9304" layer="101" font="vector">Current and Voltage Sense Module</text>
 </plain>
 <instances>
@@
 <text x="199.4662" y="19.6342" size="1.9304" layer="100" font="vector">Title</text>
 <text x="180.9242" y="19.6342" size="1.9304" layer="102" font="vector">H2AR3</text>
-<text x="179.2478" y="11.2014" size="1.9304" layer="101" font="vector">RGB LED</text>
+<text x="170.3578" y="11.2014" size="1.9304" layer="101" font="vector">Current and Voltage Sense Module</text>
 <text x="206.3242" y="19.6342" size="1.9304" layer="101" font="vector">H2AR3_Frontend</text>
 <wire x1="168.91" y1="3.81" x2="168.91" y2="8.128" width="0.1524" layer="205"/>
@@
 <text x="242.6462" y="6.1722" size="1.9304" layer="100" font="vector">www.hexabitz.com</text>
 <text x="25.4" y="198.12" size="1.778" layer="150">VDD=3.3 Volts</text>
-<text x="181.3378" y="4.9414" size="1.9304" layer="101" font="vector">Amir_Tabbakh</text>
+<text x="182.6078" y="4.9414" size="1.9304" layer="101" font="vector">Amir_Tabbakh</text>
 <text x="121.92" y="59.69" size="1.778" layer="95">U2_filter</text>
 <text x="93.98" y="59.69" size="1.778" layer="95">U3_filter</text>

Commit message: some fixes
Parts:
- R10, R9: value 330k -> 1M
- R8: value 330K -> 1M
Other:
- note added: "CT_connector"
- note added: "Voltage_connector"
Changed lines of the file:
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@@
 <part name="SUPPLY18" library="supply2" deviceset="AGND" device="" value="VSSA"/>
 <part name="SUPPLY19" library="supply2" deviceset="AGND" device="" value="VSSA"/>
-<part name="R8" library="HEXABITZ_RCLS" library_urn="urn:adsk.eagle:library:20064561" deviceset="R_1206" device="R1206" package3d_urn="urn:adsk.eagle:package:23540/2" value="330K"/>
-<part name="R9" library="HEXABITZ_RCLS" library_urn="urn:adsk.eagle:library:20064561" deviceset="R_1206" device="R1206" package3d_urn="urn:adsk.eagle:package:23540/2" value="330k"/>
-<part name="R10" library="HEXABITZ_RCLS" library_urn="urn:adsk.eagle:library:20064561" deviceset="R_1206" device="R1206" package3d_urn="urn:adsk.eagle:package:23540/2" value="330k"/>
+<part name="R8" library="HEXABITZ_RCLS" library_urn="urn:adsk.eagle:library:20064561" deviceset="R_1206" device="R1206" package3d_urn="urn:adsk.eagle:package:23540/2" value="1M"/>
+<part name="R9" library="HEXABITZ_RCLS" library_urn="urn:adsk.eagle:library:20064561" deviceset="R_1206" device="R1206" package3d_urn="urn:adsk.eagle:package:23540/2" value="1M"/>
+<part name="R10" library="HEXABITZ_RCLS" library_urn="urn:adsk.eagle:library:20064561" deviceset="R_1206" device="R1206" package3d_urn="urn:adsk.eagle:package:23540/2" value="1M"/>
 <part name="U3" library="HEXABITZ_ICs" library_urn="urn:adsk.eagle:library:20064554" deviceset="INA199A2DCKT" device="" package3d_urn="urn:adsk.eagle:package:19904117/2" value="INA199B2DCKT"/>
 <part name="C16" library="HEXABITZ_RCLS" library_urn="urn:adsk.eagle:library:20064561" deviceset="C-0603" device="" package3d_urn="urn:adsk.eagle:package:19666468/2" value="10uF"/>
@@
 <text x="93.98" y="59.69" size="1.778" layer="95">U3_filter</text>
 <text x="74.93" y="59.69" size="1.778" layer="95">U4_filter</text>
+<text x="30.48" y="66.04" size="1.778" layer="150">CT_connector</text>
+<text x="30.48" y="40.64" size="1.778" layer="150">Voltage_connector</text>
 </plain>
 <instances>

Commit message: no message
Parts:
- removed C13, C20: 1.00uF, HEXABITZ_RCLS:C-0805-POL
- C10: CAPACITANCE (none) -> 10uF; MFN (none) -> KEMET; MPN (none) -> C0603C106M9PACTU; OCTOPART_URL (none) -> https://octopart.com/c0603c106m9pactu-kemet-8375727?r=sp; VOLTAGE_RATING (none) -> 6.3v
- C11, C12, C17, C18: CAPACITANCE (none) -> 1uF; MFN (none) -> KEMET; MPN (none) -> C0603C105K8RACTU; OCTOPART_URL (none) -> https://octopart.com/c0603c105k8ractu-kemet-12595642?r=sp; TOLERANCE (none) -> 10%; VOLTAGE_RATING (none) -> 10v
- C16: CAPACITANCE (none) -> 10uF; MFN (none) -> KEMET; MPN (none) -> C0603C106M9PACTU; OCTOPART_URL (none) -> https://octopart.com/c0603c106m9pactu-kemet-8375727?r=sp; TOLERANCE (none) -> 20%; VOLTAGE_RATING (none) -> 6.3V
- FB2, FB3, FB4, FB5: MFN (none) -> Taiyo Yuden; MPN (none) -> FBMJ2125HM210NT; OCTOPART_URL (none) -> https://octopart.com/fbmj2125hm210nt-taiyo+yuden-368424?r=sp
- P1: value HEXABIT_17.32 -> HEXABIT__NO_P1_P5_P6_P7_P12; device hexabitz_connectors:HEXABIT_17.32 -> hexabitz_connectors:HEXABIT__NO_P1_P5_P6_P7_P12
- R10, R8, R9: value 1M -> 1M0; MFN (none) -> Yageo; MPN (none) -> RT1206BRD071ML; OCTOPART_URL (none) -> https://octopart.com/rt1206brd071ml-yageo-1262221?r=sp
- R11, R12, R4, R5: value 1.01R -> 1R0; MFN (none) -> Vishay; MPN (none) -> CRCW06031R00FKEA; OCTOPART_URL (none) -> https://octopart.com/crcw06031r00fkea-vishay-39713722?r=sp&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; RESISTANCE (none) -> 1; TOLERANCE (none) -> 1%
- R13, R7: MFN (none) -> Yageo; MPN (none) -> RC0603JR-071KL; OCTOPART_URL (none) -> https://octopart.com/rc0603jr-071kl-yageo-55402888?r=sp; RESISTANCE (none) -> 1K; TOLERANCE (none) -> 5%
- R14: value 3.3K -> 150R; device HEXABITZ_RCLS:R-0603 -> HEXABITZ_RCLS:R_1206R1206; MFN (none) -> Panasonic; MPN (none) -> ERA-8AEB151V; OCTOPART_URL (none) -> https://octopart.com/era-8aeb151v-panasonic-55477439?r=sp
- R15: MFN (none) -> Vishay; MPN (none) -> CRCW0603150KFKEA; OCTOPART_URL (none) -> https://octopart.com/crcw0603150kfkea-vishay-39455816?r=sp; RESISTANCE (none) -> 150K; TOLERANCE (none) -> 1%
- U2: device HEXABITZ_ICs:INA199A2DCKT -> HEXABITZ_ICs:INA199B2DCKT; MPN INA199B2DCKT -> (none)
- U3: value INA199B2DCKT -> INA199B1DCKT; device HEXABITZ_ICs:INA199A2DCKT -> HEXABITZ_ICs:INA199B1DCKT
- U4: value TEXAS_INSTRUMENTS_REF3212AIDBVRTEXAS_INSTRUMENTS_REF3212AIDBVR_0_0 -> TEXAS_INSTRUMENTS_REF2033AIDDCRTEXAS_INSTRUMENTS_REF2033AIDDCR_0_2; device HEXABITZ_ICs:TEXAS_INSTRUMENTS_REF3212AIDBVRTEXAS_INSTRUMENTS_REF3212AIDBVR_0_0 -> HEXABITZ_ICs:TEXAS_INSTRUMENTS_REF2033AIDDCRTEXAS_INSTRUMENTS_REF2033AIDDCR_0_2
Connections:
- net N$13 renamed CURRENT_P
- net N$14 renamed CURRENT_N
- removed net USART1_RX: P1.SD5, U1.PA10
- removed net USART1_TX: P1.SU5, U1.PA9
- removed net USART4_RX: P1.SD1, U1.PA1
- removed net USART4_TX: P1.SU1, U1.PA0
- removed net VDDA: C1.1, C13.+, C14.1, C2.+, C20.+, C21.1, C24.+, FB1.1, U1.VDDA
- removed net VSSA: C1.2, C13.-, C14.2, C2.-, C20.-, C21.2, C24.-, R2.2, U1.VSS_A
- net AGND: now also C1.2, C14.2, C2.-, C21.2, C24.-, R2.2, U1.VSS_A, U4.GND; no longer U4.GND_F, U4.GND_S
- net CURRENT_SENSE: now also U1.PA7; no longer U1.PA8
- net GND: now also U1.PB14, U1.PB15, U1.PB2, U1.PC13, U1.PC14-OSC32_IN; no longer P1.GND1, P1.GND6
- net N$16: now also U4.EN; no longer U4.ENABLE
- net NEUTRAL: now also P2.1; no longer P2.2
- net PHASE: now also P2.2; no longer P2.1
- net USART5_RX: no longer P1.SD6
- net USART5_TX: no longer P1.SU6
- net VCC: now also C1.1, C14.1, C2.+, C21.1, C24.+, FB1.1, U1.VDDA, U4.VIN, U4.VREF; no longer U4.IN
- net VDD: no longer P1.VDD1, P1.VDD6
- net VOLTAGE_SENSE: now also U1.PA8; no longer U1.PA7
- net V_REF: now also U4.VBIAS; no longer U4.OUT_F, U4.OUT_S
Other:
- note added: "Gain = 50 V/V"
- note added: "Gain= 100 V/V"
- note added: "V_ref = 1.65V"
- moved on the sheet: C22, C23, R15, U2
